File: KiCad/gluhwurmchen/gluhwurmchen.kicad_pcb (KiCad board)
At the start: 2 copper layers, 30.6 x 30.6 mm, 13 parts, among them J1 3V_ext, J2 GND_ext, Q1 2N3904, U1 CR2032

Commit message: changed trough-hole to smd
Parts:
- D1: footprint gluhwurmchen:LED_D5.0mm_handsolder -> LED_SMD:LED_0603_1608Metric_Pad1.05x0.95mm_HandSolder
- Q1: footprint gluhwurmchen:TO-92L_Inline_Handsolder -> Package_TO_SOT_SMD:SOT-23
- R1: footprint gluhwurmchen:R_Axial_12.7mm_handsolder -> Resistor_SMD:R_0603_1608Metric_Pad0.98x0.95mm_HandSolder
- moved R1 9.61 mm to (76.2, 89.5), turned to -90 degrees
- moved REF** 9.24 mm to (83.3, 91.4), turned to 0 degrees
- moved Q1 7.18 mm to (83.8, 96.5), turned to 180 degrees
- moved D1 0.63 mm to (87.0, 88.9), turned to -90 degrees
Routing:
- net (no net): track 97.3 -> 0.00 mm
- net Net-(D1-K): track 64.0 -> 42.1 mm
- net Net-(D2-C): track 36.7 -> 29.3 mm
- net Net-(D1-A): track 7.40 -> 9.50 mm
- net Net-(J1-Pin_1): track 45.0 -> 45.8 mm
Other:
- board text removed: "wienXtra"
